Commit message: Increase magnitude of robot, refactoring code (needed params are arguments)

File: strirus_robot_description/urdf/strirus.xacro (robot description, xacro)
@@ -7,25 +7,32 @@
 	<xacro:property name="deg2rad" value="${pi / 180}" />
 	<!-- Constants for simulating -->
-	<!-- number of legs need to be real number - 1 -->
-	<xacro:property name="real_number_of_legs" value="19" />
+	<!-- number of legs need to be real number - 1 (it is from one side only)-->
+	<!-- Xacro arg provides xacro.py file.xacro real_number_of_legs:=3 -->
+	<xacro:arg name="real_number_of_legs" default="6" />
+	<xacro:arg name="angle_between_legs" default="90" />
+	<!-- in degree -->
+	<xacro:arg name="offset_between_legs_wave" default="0" />
+	<!-- scale is needed for easily change scale of stl -->
+	<xacro:property name="scale" value="5" />
+	<xacro:property name="real_number_of_legs" value="$(arg real_number_of_legs)" />
 	<xacro:property name="number_of_legs" value="${real_number_of_legs - 1}" />
-	<xacro:property name="angle_between_legs" value="60" />
+	<xacro:property name="angle_between_legs" value="$(arg angle_between_legs)" />
 	<!-- in degree -->
-	<xacro:property name="offset_between_legs_wave" value="0" />
+	<xacro:property name="offset_between_legs_wave" value="$(arg offset_between_legs_wave)" />
 	<!-- Body and leg Constants -->
-	<xacro:property name="body_x_offset" value="0" />
+	<xacro:property name="body_x_offset" value="${0 * scale}" />
 	<xacro:property name="body_y_offset" value="${body_length / 2}" />
 	<xacro:property name="body_z_offset" value="${leg_width + leg_height}" />
-	<xacro:property name="first_hole_x_offset" value="0.05" />
-	<xacro:property name="body_width" value="0.5" />
-	<xacro:property name="body_height" value="0.07" />
-	<xacro:property name="body_weight" value="${body_width * body_length * body_height * 250}"/>
-	<xacro:property name="leg_x_offset" value="0" />
-	<xacro:property name="leg_y_offset" value="0" />
-	<xacro:property name="leg_z_offset" value="0" />
-	<xacro:property name="leg_x_offset_in_body" value="-0.075" />
-	<xacro:property name="leg_width" value="0.02" />
-	<xacro:property name="leg_height" value="0.08" />
-	<xacro:property name="fallibility_between_legs" value="${0.002 + 2 * leg_width}" />
+	<xacro:property name="first_hole_x_offset" value="${0.05 * scale}" />
+	<xacro:property name="body_width" value="${0.5 * scale}" />
+	<xacro:property name="body_height" value="${0.07 * scale}" />
+	<xacro:property name="body_weight" value="${body_width * body_length * body_height * 0.3}"/>
+	<xacro:property name="leg_x_offset" value="${0 * scale}" />
+	<xacro:property name="leg_y_offset" value="${0 * scale}" />
+	<xacro:property name="leg_z_offset" value="${0 * scale}" />
+	<xacro:property name="leg_x_offset_in_body" value="${-0.075 * scale}" />
+	<xacro:property name="leg_width" value="${0.02 * scale}" />
+	<xacro:property name="leg_height" value="${0.08 * scale}" />
+	<xacro:property name="fallibility_between_legs" value="${(0.002 * scale) + 2 * leg_width}" />
 	<!-- Formulas -->
 	<xacro:property name="dist_between_legs" value="${leg_height * sin(angle_between_legs * deg2rad) + fallibility_between_legs}" />
@@ -35,7 +42,7 @@
 		<link name="leg_${prefix}_${num}">
 			<inertial>
-				<mass value="0.00035"/>
+				<mass value="${0.05 * scale}"/>
 				<origin rpy="0  0  0" xyz="${leg_x_offset} ${leg_y_offset} ${leg_z_offset}"/>
-				<inertia ixx="0.0001" ixy="0" ixz="0" iyy="0.0001" iyz="0" izz="0.0001"/>
+				<inertia ixx="0.001" ixy="0" ixz="0" iyy="0.001" iyz="0" izz="0.001"/>
 			</inertial>
 			<collision >
@@ -48,5 +55,5 @@
 				</xacro:if>
 				<geometry>
-					<mesh filename="package://strirus_robot_description/meshes/stl/leg_30_degree.stl" scale="1.0 1.0 1.0"/>
+					<mesh filename="package://strirus_robot_description/meshes/stl/leg_30_degree_normal.stl" scale="1.0 1.0 1.0"/>
 				</geometry>
 			</collision>
@@ -59,5 +66,5 @@
 				</xacro:if>
 				<geometry>
-					<mesh filename="package://strirus_robot_description/meshes/stl/leg_30_degree.stl" scale="1.0 1.0 1.0"/>
+					<mesh filename="package://strirus_robot_description/meshes/stl/leg_30_degree_normal.stl" scale="1.0 1.0 1.0"/>
 				</geometry>
 				<material name="blue"/>
@@ -68,7 +75,8 @@
 		<parent link="body"/>
 			<child link="leg_${prefix}_${num}"/>
-			<origin rpy="0       0      0" xyz="${(body_width / 4 + leg_x_offset_in_body)* side} ${first_hole_x_offset + (num) * dist_between_legs}  ${body_z_offset}"/>
+			<origin rpy="0       0      0" xyz="${(body_width / 4 + leg_x_offset_in_body) * side} ${first_hole_x_offset + (num) * dist_between_legs}  ${body_z_offset}"/>
 			<axis xyz="1 0  0"/>
-			<limit effort="-1" lower="-1e+100" upper="1e+100" velocity="100"/>
+			<limit effort="30" lower="-1e+100" upper="1e+100" velocity="1"/>
+			<joint_properties damping="0.0" friction="0.0" />
 		</joint>
 <!-- /////////////// -->
@@ -78,7 +86,7 @@
 				<hardwareInterface>EffortJointInterface</hardwareInterface>
 			</joint>
-			<actuator name="leg_${prefix}_${num}_actuator">
+			<actuator name="leg_${prefix}_0_actuator">
 				<hardwareInterface>EffortJointInterface</hardwareInterface>
-				<mechanicalReduction>1</mechanicalReduction>
+				<mechanicalReduction>50</mechanicalReduction>
 			</actuator>
 		</transmission>
@@ -122,13 +130,35 @@
     	</xacro:if>
 	</xacro:macro>
-<!-- create needed number of joints between legs (is implemented by recurcion)
-	<xacro:macro name="create_revolute_joints" params="prefix side number">
-    	<xacro:wheel prefix="${prefix}" num="${number}" side="${side}"/>
-    	<xacro:if value="${number}">
-        	<xacro:loop number="${number-1}" prefix="${prefix}" side="${side}"/>
+<!-- create needed number of joints between legs (is implemented by recurcion) -->
+<!-- 	<xacro:macro name="create_dependence_between_legs" params="prefix side number">
+    			<joint name="legs_${prefix}_${number}_and_${number - 1}_revolute_joint" type="revolute">
+		<parent link="leg_${prefix}_${number}"/>
+			<child link="leg_${prefix}_${number - 1}"/>
+			<origin rpy="0       0      0" xyz="0 ${-dist_between_legs} 0"/>
+			<axis xyz="1 0  0"/>
+			<limit effort="-1" lower="-1e+100" upper="1e+100" velocity="100"/>
+		</joint>
+    	<xacro:if value="${number - 1}">
+        	<xacro:create_dependence_between_legs number="${number-1}" prefix="${prefix}" side="${side}"/>
     	</xacro:if>
-	</xacro:macro>
--->
+	</xacro:macro> -->
 <xacro:create_legs prefix="left" side="1" number="${number_of_legs}" />
 <xacro:create_legs prefix="right" side="-1" number="${number_of_legs}" />
+<!-- <xacro:create_dependence_between_legs prefix="left" side="1" number="${number_of_legs}" />
+<xacro:create_dependence_between_legs prefix="right" side="-1" number="${number_of_legs}" /> -->
+<!--  <joint name="legs_l_1_and_0_revolute_joint" type="fixed">
+		<parent link="leg_left_0"/>
+			<child link="leg_left_1"/>
+			<origin rpy="0  0  0" xyz="0 ${dist_between_legs} 0"/>
+			<axis xyz="0 0  0"/>
+			<limit effort="40" lower="-1e+100" upper="1e+100" velocity="3"/>
+		</joint>
+ <joint name="legs_r_1_and_0_revolute_joint" type="fixed">
+		<parent link="leg_right_0"/>
+			<child link="leg_right_1"/>
+			<origin rpy="0  0  0" xyz="0 ${dist_between_legs} 0"/>
+			<axis xyz="0 0  0"/>
+			<limit effort="40" lower="-1e+100" upper="1e+100" velocity="3"/>
+		</joint>
+  -->
 </robot>

Commit message: fix bug with body's collision

File: strirus_robot_description/urdf/strirus.xacro (robot description, xacro)
@@ -112,5 +112,5 @@
 			<origin rpy="0  0  0" xyz="${body_x_offset} ${body_y_offset}  ${body_z_offset}"/>
 			<geometry>
-				<box size="${body_width / 2} ${body_length /2} ${body_height / 2}"/>
+				<box size="${body_width / 2} ${body_length} ${body_height / 2}"/>
 			</geometry>
 		</collision>

Commit message: Example works in rviz with state_publisher, but without gazebo

File: strirus_robot_description/urdf/strirus.xacro (robot description, xacro)
@@ -9,6 +9,6 @@
 	<!-- number of legs need to be real number - 1 (it is from one side only)-->
 	<!-- Xacro arg provides xacro.py file.xacro real_number_of_legs:=3 -->
-	<xacro:arg name="real_number_of_legs" default="6" />
-	<xacro:arg name="angle_between_legs" default="90" />
+	<xacro:arg name="real_number_of_legs" default="5" />
+	<xacro:arg name="angle_between_legs" default="89" />
 	<!-- in degree -->
 	<xacro:arg name="offset_between_legs_wave" default="0" />
@@ -42,15 +42,15 @@
 		<link name="leg_${prefix}_${num}">
 			<inertial>
-				<mass value="${0.05 * scale}"/>
+				<mass value="${0.01 * scale}"/>
 				<origin rpy="0  0  0" xyz="${leg_x_offset} ${leg_y_offset} ${leg_z_offset}"/>
-				<inertia ixx="0.001" ixy="0" ixz="0" iyy="0.001" iyz="0" izz="0.001"/>
+				<inertia ixx="0.0" ixy="0" ixz="0" iyy="0.00" iyz="0" izz="0.00"/>
 			</inertial>
 			<collision >
-			<!-- legs wave offset change only on the left side -->
+				<!-- legs wave offset change only on the left side -->
 				<xacro:if value="${prefix == 'left'}">
-				<origin rpy="${(offset_between_legs_wave + angle_between_legs * num) % 360 * deg2rad} 0 0" xyz="${leg_x_offset} ${leg_y_offset} ${leg_z_offset}"/>
+					<origin rpy="${(offset_between_legs_wave + angle_between_legs * num) % 360 * deg2rad} 0 0" xyz="${leg_x_offset} ${leg_y_offset} ${leg_z_offset}"/>
 				</xacro:if>
 				<xacro:if value="${prefix == 'right'}">
-				<origin rpy="${-(angle_between_legs * num) % 360 * deg2rad} 0 ${pi}" xyz="${leg_x_offset} ${leg_y_offset} ${leg_z_offset}"/>
+					<origin rpy="${-(angle_between_legs * num) % 360 * deg2rad} 0 ${pi}" xyz="${leg_x_offset} ${leg_y_offset} ${leg_z_offset}"/>
 				</xacro:if>
 				<geometry>
@@ -60,8 +60,8 @@
 			<visual>
 				<xacro:if value="${prefix == 'left'}">
-				<origin rpy="${(offset_between_legs_wave + angle_between_legs * num) % 360 * deg2rad} 0 0" xyz="${leg_x_offset} ${leg_y_offset} ${leg_z_offset}"/>
+					<origin rpy="${(offset_between_legs_wave + angle_between_legs * num) % 360 * deg2rad} 0 0" xyz="${leg_x_offset} ${leg_y_offset} ${leg_z_offset}"/>
 				</xacro:if>
 				<xacro:if value="${prefix == 'right'}">
-				<origin rpy="${-(angle_between_legs * num) % 360 * deg2rad} 0 ${pi}" xyz="${leg_x_offset} ${leg_y_offset} ${leg_z_offset}"/>
+					<origin rpy="${-(angle_between_legs * num) % 360 * deg2rad} 0 ${pi}" xyz="${leg_x_offset} ${leg_y_offset} ${leg_z_offset}"/>
 				</xacro:if>
 				<geometry>
@@ -71,15 +71,15 @@
 			</visual>
 		</link>
-<!-- /////////////// -->
-		<joint name="leg_${prefix}_${num}_revolute_joint" type="revolute">
+		<!-- /////////////// -->
+<!-- 		<joint name="leg_${prefix}_${num}_revolute_joint" type="revolute">
 		<parent link="body"/>
 			<child link="leg_${prefix}_${num}"/>
 			<origin rpy="0       0      0" xyz="${(body_width / 4 + leg_x_offset_in_body) * side} ${first_hole_x_offset + (num) * dist_between_legs}  ${body_z_offset}"/>
 			<axis xyz="1 0  0"/>
-			<limit effort="30" lower="-1e+100" upper="1e+100" velocity="1"/>
-			<joint_properties damping="0.0" friction="0.0" />
-		</joint>
-<!-- /////////////// -->
-		<transmission name="leg_${prefix}_${num}_transmission">
+			<limit effort="30" lower="-1e+100" upper="1e+100" velocity="3"/>
+			<joint_properties damping="900.0" friction="900.0" />
+		</joint> -->
+		<!-- /////////////// -->
+<!-- 		<transmission name="leg_${prefix}_${num}_transmission">
 			<type>transmission_interface/SimpleTransmission</type>
 			<joint name="leg_${prefix}_${num}_revolute_joint">
@@ -91,21 +91,77 @@
 			</actuator>
 		</transmission>
+	-->
+</xacro:macro>
+	<!-- create needed number of legs (is implemented by recurcion) -->
+<!-- 	<xacro:macro name="create_legs" params="prefix side number">
+		<xacro:leg prefix="${prefix}" num="${number}" side="${side}"/>
+		<xacro:if value="${number}">
+			<xacro:create_legs number="${number-1}" prefix="${prefix}" side="${side}"/>
+		</xacro:if>
 	</xacro:macro>
-	<!-- Body description -->
-	<link name="base_link"/>
-	<joint name="base_link_body_fixed" type="fixed">
-	    <parent link="base_link"/>
-	    <child link="body"/>
-	</joint>
+    <xacro:create_legs prefix="left" side="1" number="${number_of_legs}" />
+ -->
+ 	<xacro:leg prefix="left" num="0" side="1"/>
+ 	<xacro:leg prefix="left" num="1" side="1"/>
+ 	<xacro:leg prefix="left" num="2" side="1"/>
+ 	<xacro:leg prefix="left" num="3" side="1"/>
+ 	<xacro:leg prefix="left" num="4" side="1"/>
+    <joint name="leg_left_0_revolute_joint" type="revolute">
+	<parent link="body"/>
+	<child link="leg_left_0"/>
+	<origin rpy="0       0      0" xyz="${(body_width / 4 + leg_x_offset_in_body) * 1} ${first_hole_x_offset + (0) * dist_between_legs}  ${body_z_offset}"/>
+	<axis xyz="1 0  0"/>
+	<limit effort="30" lower="-1e+100" upper="1e+100" velocity="3"/>
+</joint>
+<joint name="leg_left_1_revolute_joint" type="revolute">
+	<parent link="body"/>
+	<child link="leg_left_1"/>
+	<origin rpy="0       0      0" xyz="${(body_width / 4 + leg_x_offset_in_body) * 1} ${first_hole_x_offset + (1) * dist_between_legs}  ${body_z_offset}"/>
+	<axis xyz="1 0  0"/>
+	<limit effort="30" lower="-1e+100" upper="1e+100" velocity="3"/>
+	<mimic joint="leg_left_0_revolute_joint" multiplier="1" offset="0" />
+</joint>
+<joint name="leg_left_2_revolute_joint" type="revolute">
+	<parent link="body"/>
+	<child link="leg_left_2"/>
+	<origin rpy="0       0      0" xyz="${(body_width / 4 + leg_x_offset_in_body) * 1} ${first_hole_x_offset + (2) * dist_between_legs}  ${body_z_offset}"/>
+	<axis xyz="1 0  0"/>
+	<limit effort="30" lower="-1e+100" upper="1e+100" velocity="3"/>
+	<mimic joint="leg_left_0_revolute_joint" multiplier="1" offset="0" />
+</joint>
+<joint name="leg_left_3_revolute_joint" type="revolute">
+	<parent link="body"/>
+	<child link="leg_left_3"/>
+	<origin rpy="0       0      0" xyz="${(body_width / 4 + leg_x_offset_in_body) * 1} ${first_hole_x_offset + (3) * dist_between_legs}  ${body_z_offset}"/>
+	<axis xyz="1 0  0"/>
+	<limit effort="30" lower="-1e+100" upper="1e+100" velocity="3"/>
+	<mimic joint="leg_left_0_revolute_joint" multiplier="1" offset="0" />
+</joint>
+<joint name="leg_left_4_revolute_joint" type="revolute">
+	<parent link="body"/>
+	<child link="leg_left_4"/>
+	<origin rpy="0       0      0" xyz="${(body_width / 4 + leg_x_offset_in_body) * 1} ${first_hole_x_offset + (4) * dist_between_legs}  ${body_z_offset}"/>
+	<axis xyz="1 0  0"/>
+	<limit effort="30" lower="-1e+100" upper="1e+100" velocity="3"/>
+	<mimic joint="leg_left_0_revolute_joint" multiplier="1" offset="0" />
+</joint>
+<!-- Body description -->
+<link name="base_link"/>
+<joint name="base_link_body_fixed" type="fixed">
+	<parent link="base_link"/>
+	<child link="body"/>
+</joint>
 <!-- /////////////// -->
-	<link name="body">
-		<inertial>
-			<!-- 250 value is mass density, the value is just empiric-->
-			<mass value="${body_weight}"/>
-			<origin rpy="0  0  0" xyz="${body_x_offset} ${body_y_offset}  ${body_z_offset}"/>
-			<inertia
+<link name="body">
+	<inertial>
+		<!-- 250 value is mass density, the value is just empiric-->
+		<mass value="${body_weight}"/>
+		<origin rpy="0  0  0" xyz="${body_x_offset} ${body_y_offset}  ${body_z_offset}"/>
+<!--			<inertia
 				ixx="${1/12 * body_weight * (body_height * body_height + body_length * body_length)}"  ixy="0"  ixz="0"
 				iyy="${1/12 * body_weight * (body_height * body_height + body_width * body_width)}" iyz="0"
 				izz="${1/12 * body_weight * (body_length * body_length + body_width * body_width)}" />
+			-->
+			<inertia ixx="0.0" ixy="0" ixz="0" iyy="0.00" iyz="0" izz="0.00"/>
 		</inertial>
 		<collision >
@@ -123,12 +179,5 @@
 		</visual>
 	</link>
-<!-- create needed number of legs (is implemented by recurcion) -->
-	<xacro:macro name="create_legs" params="prefix side number">
-    	<xacro:leg prefix="${prefix}" num="${number}" side="${side}"/>
-    	<xacro:if value="${number}">
-        	<xacro:create_legs number="${number-1}" prefix="${prefix}" side="${side}"/>
-    	</xacro:if>
-	</xacro:macro>
-<!-- create needed number of joints between legs (is implemented by recurcion) -->
+	<!-- create needed number of joints between legs (is implemented by recurcion) -->
 <!-- 	<xacro:macro name="create_dependence_between_legs" params="prefix side number">
     			<joint name="legs_${prefix}_${number}_and_${number - 1}_revolute_joint" type="revolute">
@@ -142,23 +191,32 @@
         	<xacro:create_dependence_between_legs number="${number-1}" prefix="${prefix}" side="${side}"/>
     	</xacro:if>
-	</xacro:macro> -->
-<xacro:create_legs prefix="left" side="1" number="${number_of_legs}" />
-<xacro:create_legs prefix="right" side="-1" number="${number_of_legs}" />
-<!-- <xacro:create_dependence_between_legs prefix="left" side="1" number="${number_of_legs}" />
-<xacro:create_dependence_between_legs prefix="right" side="-1" number="${number_of_legs}" /> -->
-<!--  <joint name="legs_l_1_and_0_revolute_joint" type="fixed">
-		<parent link="leg_left_0"/>
-			<child link="leg_left_1"/>
-			<origin rpy="0  0  0" xyz="0 ${dist_between_legs} 0"/>
-			<axis xyz="0 0  0"/>
-			<limit effort="40" lower="-1e+100" upper="1e+100" velocity="3"/>
-		</joint>
- <joint name="legs_r_1_and_0_revolute_joint" type="fixed">
-		<parent link="leg_right_0"/>
-			<child link="leg_right_1"/>
-			<origin rpy="0  0  0" xyz="0 ${dist_between_legs} 0"/>
-			<axis xyz="0 0  0"/>
-			<limit effort="40" lower="-1e+100" upper="1e+100" velocity="3"/>
-		</joint>
-  -->
+    </xacro:macro> -->
+    <!-- <xacro:create_legs prefix="right" side="-1" number="${number_of_legs}" /> -->
+<!--
+	<joint type="revolute" name="legs_left_0_and_1_revolute_joint">
+      <pose>0 ${-dist_between_legs} 0 0 0 0</pose>
+      <parent>leg_left_0</parent>
+      <child>leg_left_1</child>
+      <axis>
+        <xyz>1 0 0</xyz>
+      </axis>
+  </joint> -->
+<!-- <gazebo>
+	<joint type="revolute" name="legs_left_0_and_1_revolute_joint">
+      <pose>0 ${-dist_between_legs} 0 0 0 0</pose>
+      <parent>leg_left_0</parent>
+      <child>leg_left_1</child>
+      <axis>
+        <xyz>1 0 0</xyz>
+      </axis>
+    </joint>
+    	<joint type="revolute" name="legs_left_1_and_0_revolute_joint">
+      <pose>0 ${dist_between_legs} 0 0 0 0</pose>
+      <parent>leg_left_1</parent>
+      <child>leg_left_0</child>
+      <axis>
+        <xyz>1 0 0</xyz>
+      </axis>
+    </joint>
+</gazebo> -->
 </robot>
