Commit message: robot move statisfactory but with some troubles

File: strirus_robot_description/urdf/strirus.xacro (robot description, xacro)
@@ -9,6 +9,6 @@
 	<!-- number of legs need to be real number - 1 (it is from one side only)-->
 	<!-- Xacro arg provides xacro.py file.xacro real_number_of_legs:=3 -->
-	<xacro:arg name="real_number_of_legs" default="5" />
-	<xacro:arg name="angle_between_legs" default="89" />
+	<xacro:arg name="real_number_of_legs" default="19" />
+	<xacro:arg name="angle_between_legs" default="60" />
 	<!-- in degree -->
 	<xacro:arg name="offset_between_legs_wave" default="0" />
@@ -42,7 +42,7 @@
 		<link name="leg_${prefix}_${num}">
 			<inertial>
-				<mass value="${0.01 * scale}"/>
+				<mass value="${0.05 * scale}"/>
 				<origin rpy="0  0  0" xyz="${leg_x_offset} ${leg_y_offset} ${leg_z_offset}"/>
-				<inertia ixx="0.0" ixy="0" ixz="0" iyy="0.00" iyz="0" izz="0.00"/>
+				<inertia ixx="0.001" ixy="0" ixz="0" iyy="0.001" iyz="0" izz="0.001"/>
 			</inertial>
 			<collision >
@@ -72,14 +72,14 @@
 		</link>
 		<!-- /////////////// -->
-<!-- 		<joint name="leg_${prefix}_${num}_revolute_joint" type="revolute">
-		<parent link="body"/>
+		<joint name="leg_${prefix}_${num}_revolute_joint" type="revolute">
+			<parent link="body"/>
 			<child link="leg_${prefix}_${num}"/>
 			<origin rpy="0       0      0" xyz="${(body_width / 4 + leg_x_offset_in_body) * side} ${first_hole_x_offset + (num) * dist_between_legs}  ${body_z_offset}"/>
 			<axis xyz="1 0  0"/>
 			<limit effort="30" lower="-1e+100" upper="1e+100" velocity="3"/>
-			<joint_properties damping="900.0" friction="900.0" />
-		</joint> -->
+			<joint_properties damping="0.0" friction="0.0" />
+		</joint>
 		<!-- /////////////// -->
- 		<transmission name="leg_${prefix}_${num}_transmission">
+		<transmission name="leg_${prefix}_${num}_transmission">
 			<type>transmission_interface/SimpleTransmission</type>
 			<joint name="leg_${prefix}_${num}_revolute_joint">
@@ -91,131 +91,44 @@
 			</actuator>
 		</transmission>
-</xacro:macro>
-	<!-- create needed number of legs (is implemented by recurcion) -->
-<!-- 	<xacro:macro name="create_legs" params="prefix side number">
-		<xacro:leg prefix="${prefix}" num="${number}" side="${side}"/>
-		<xacro:if value="${number}">
-			<xacro:create_legs number="${number-1}" prefix="${prefix}" side="${side}"/>
-		</xacro:if>
 	</xacro:macro>
-    <xacro:create_legs prefix="left" side="1" number="${number_of_legs}" />
- -->
- 	<xacro:leg prefix="left" num="0" side="1"/>
- 	<xacro:leg prefix="left" num="1" side="1"/>
- 	<xacro:leg prefix="left" num="2" side="1"/>
- 	<xacro:leg prefix="left" num="3" side="1"/>
- 	<xacro:leg prefix="left" num="4" side="1"/>
-    <joint name="leg_left_0_revolute_joint" type="revolute">
-	<parent link="body"/>
-	<child link="leg_left_0"/>
-	<origin rpy="0       0      0" xyz="${(body_width / 4 + leg_x_offset_in_body) * 1} ${first_hole_x_offset + (0) * dist_between_legs}  ${body_z_offset}"/>
-	<axis xyz="1 0  0"/>
-	<limit effort="30" lower="-1e+100" upper="1e+100" velocity="3"/>
-</joint>
-<joint name="leg_left_1_revolute_joint" type="revolute">
-	<parent link="body"/>
-	<child link="leg_left_1"/>
-	<origin rpy="0       0      0" xyz="${(body_width / 4 + leg_x_offset_in_body) * 1} ${first_hole_x_offset + (1) * dist_between_legs}  ${body_z_offset}"/>
-	<axis xyz="1 0  0"/>
-	<limit effort="30" lower="-1e+100" upper="1e+100" velocity="3"/>
-	<mimic joint="leg_left_0_revolute_joint" multiplier="1" offset="0" />
-</joint>
-<joint name="leg_left_2_revolute_joint" type="revolute">
-	<parent link="body"/>
-	<child link="leg_left_2"/>
-	<origin rpy="0       0      0" xyz="${(body_width / 4 + leg_x_offset_in_body) * 1} ${first_hole_x_offset + (2) * dist_between_legs}  ${body_z_offset}"/>
-	<axis xyz="1 0  0"/>
-	<limit effort="30" lower="-1e+100" upper="1e+100" velocity="3"/>
-	<mimic joint="leg_left_0_revolute_joint" multiplier="1" offset="0" />
-</joint>
-<joint name="leg_left_3_revolute_joint" type="revolute">
-	<parent link="body"/>
-	<child link="leg_left_3"/>
-	<origin rpy="0       0      0" xyz="${(body_width / 4 + leg_x_offset_in_body) * 1} ${first_hole_x_offset + (3) * dist_between_legs}  ${body_z_offset}"/>
-	<axis xyz="1 0  0"/>
-	<limit effort="30" lower="-1e+100" upper="1e+100" velocity="3"/>
-	<mimic joint="leg_left_0_revolute_joint" multiplier="1" offset="0" />
-</joint>
-<joint name="leg_left_4_revolute_joint" type="revolute">
-	<parent link="body"/>
-	<child link="leg_left_4"/>
-	<origin rpy="0       0      0" xyz="${(body_width / 4 + leg_x_offset_in_body) * 1} ${first_hole_x_offset + (4) * dist_between_legs}  ${body_z_offset}"/>
-	<axis xyz="1 0  0"/>
-	<limit effort="30" lower="-1e+100" upper="1e+100" velocity="3"/>
-	<mimic joint="leg_left_0_revolute_joint" multiplier="1" offset="0" />
-</joint>
-<!-- Body description -->
-<link name="base_link"/>
-<joint name="base_link_body_fixed" type="fixed">
-	<parent link="base_link"/>
-	<child link="body"/>
-</joint>
-<!-- /////////////// -->
-<link name="body">
-	<inertial>
-		<!-- 250 value is mass density, the value is just empiric-->
-		<mass value="${body_weight}"/>
-		<origin rpy="0  0  0" xyz="${body_x_offset} ${body_y_offset}  ${body_z_offset}"/>
-<!--			<inertia
+	<!-- Body description -->
+	<link name="base_link"/>
+	<joint name="base_link_body_fixed" type="fixed">
+		<parent link="base_link"/>
+		<child link="body"/>
+	</joint>
+	<!-- /////////////// -->
+	<link name="body">
+		<inertial>
+			<!-- 250 value is mass density, the value is just empiric-->
+			<mass value="${body_weight}"/>
+			<origin rpy="0  0  0" xyz="${body_x_offset} ${body_y_offset}  ${body_z_offset}"/>
+			<inertia
 				ixx="${1/12 * body_weight * (body_height * body_height + body_length * body_length)}"  ixy="0"  ixz="0"
 				iyy="${1/12 * body_weight * (body_height * body_height + body_width * body_width)}" iyz="0"
 				izz="${1/12 * body_weight * (body_length * body_length + body_width * body_width)}" />
-			-->
-			<inertia ixx="0.0" ixy="0" ixz="0" iyy="0.00" iyz="0" izz="0.00"/>
-		</inertial>
-		<collision >
-			<origin rpy="0  0  0" xyz="${body_x_offset} ${body_y_offset}  ${body_z_offset}"/>
-			<geometry>
-				<box size="${body_width / 2} ${body_length} ${body_height / 2}"/>
-			</geometry>
-		</collision>
-		<visual >
-			<origin rpy="0  0  0" xyz="${body_x_offset} ${body_y_offset}  ${body_z_offset}"/>
-			<geometry>
-				<box size="${body_width / 2} ${body_length} ${body_height / 2}"/>
-			</geometry>
-			<material name="green"/>
-		</visual>
-	</link>
-	<!-- create needed number of joints between legs (is implemented by recurcion) -->
-<!-- 	<xacro:macro name="create_dependence_between_legs" params="prefix side number">
-    			<joint name="legs_${prefix}_${number}_and_${number - 1}_revolute_joint" type="revolute">
-		<parent link="leg_${prefix}_${number}"/>
-			<child link="leg_${prefix}_${number - 1}"/>
-			<origin rpy="0       0      0" xyz="0 ${-dist_between_legs} 0"/>
-			<axis xyz="1 0  0"/>
-			<limit effort="-1" lower="-1e+100" upper="1e+100" velocity="100"/>
-		</joint>
-    	<xacro:if value="${number - 1}">
-        	<xacro:create_dependence_between_legs number="${number-1}" prefix="${prefix}" side="${side}"/>
-    	</xacro:if>
-    </xacro:macro> -->
-    <!-- <xacro:create_legs prefix="right" side="-1" number="${number_of_legs}" /> -->
-<!--
-	<joint type="revolute" name="legs_left_0_and_1_revolute_joint">
-      <pose>0 ${-dist_between_legs} 0 0 0 0</pose>
-      <parent>leg_left_0</parent>
-      <child>leg_left_1</child>
-      <axis>
-        <xyz>1 0 0</xyz>
-      </axis>
-  </joint> -->
-<!-- <gazebo>
-	<joint type="revolute" name="legs_left_0_and_1_revolute_joint">
-      <pose>0 ${-dist_between_legs} 0 0 0 0</pose>
-      <parent>leg_left_0</parent>
-      <child>leg_left_1</child>
-      <axis>
-        <xyz>1 0 0</xyz>
-      </axis>
-    </joint>
-    	<joint type="revolute" name="legs_left_1_and_0_revolute_joint">
-      <pose>0 ${dist_between_legs} 0 0 0 0</pose>
-      <parent>leg_left_1</parent>
-      <child>leg_left_0</child>
-      <axis>
-        <xyz>1 0 0</xyz>
-      </axis>
-    </joint>
-</gazebo> -->
-</robot>
+			</inertial>
+			<collision >
+				<origin rpy="0  0  0" xyz="${body_x_offset} ${body_y_offset}  ${body_z_offset}"/>
+				<geometry>
+					<box size="${body_width / 2} ${body_length} ${body_height / 2}"/>
+				</geometry>
+			</collision>
+			<visual >
+				<origin rpy="0  0  0" xyz="${body_x_offset} ${body_y_offset}  ${body_z_offset}"/>
+				<geometry>
+					<box size="${body_width / 2} ${body_length} ${body_height / 2}"/>
+				</geometry>
+				<material name="green"/>
+			</visual>
+		</link>
+		<!-- create needed number of legs (is implemented by recurcion) -->
+		<xacro:macro name="create_legs" params="prefix side number">
+			<xacro:leg prefix="${prefix}" num="${number}" side="${side}"/>
+			<xacro:if value="${number}">
+				<xacro:create_legs number="${number-1}" prefix="${prefix}" side="${side}"/>
+			</xacro:if>
+		</xacro:macro>
+		<xacro:create_legs prefix="left" side="1" number="${number_of_legs}" />
+		<xacro:create_legs prefix="right" side="-1" number="${number_of_legs}" />
+	</robot>

Commit message: refactoring code in description package

File: strirus_robot_description/urdf/strirus.xacro (robot description, xacro)
@@ -9,6 +9,6 @@
 	<!-- number of legs need to be real number - 1 (it is from one side only)-->
 	<!-- Xacro arg provides xacro.py file.xacro real_number_of_legs:=3 -->
-	<xacro:arg name="real_number_of_legs" default="6" />
-	<xacro:arg name="angle_between_legs" default="90" />
+	<xacro:arg name="real_number_of_legs" default="19" />
+	<xacro:arg name="angle_between_legs" default="60" />
 	<!-- in degree -->
 	<xacro:arg name="offset_between_legs_wave" default="0" />
@@ -47,10 +47,10 @@
 			</inertial>
 			<collision >
-			<!-- legs wave offset change only on the left side -->
+				<!-- legs wave offset change only on the left side -->
 				<xacro:if value="${prefix == 'left'}">
-				<origin rpy="${(offset_between_legs_wave + angle_between_legs * num) % 360 * deg2rad} 0 0" xyz="${leg_x_offset} ${leg_y_offset} ${leg_z_offset}"/>
+					<origin rpy="${(offset_between_legs_wave + angle_between_legs * num) % 360 * deg2rad} 0 0" xyz="${leg_x_offset} ${leg_y_offset} ${leg_z_offset}"/>
 				</xacro:if>
 				<xacro:if value="${prefix == 'right'}">
-				<origin rpy="${-(angle_between_legs * num) % 360 * deg2rad} 0 ${pi}" xyz="${leg_x_offset} ${leg_y_offset} ${leg_z_offset}"/>
+					<origin rpy="${-(angle_between_legs * num) % 360 * deg2rad} 0 ${pi}" xyz="${leg_x_offset} ${leg_y_offset} ${leg_z_offset}"/>
 				</xacro:if>
 				<geometry>
@@ -60,8 +60,8 @@
 			<visual>
 				<xacro:if value="${prefix == 'left'}">
-				<origin rpy="${(offset_between_legs_wave + angle_between_legs * num) % 360 * deg2rad} 0 0" xyz="${leg_x_offset} ${leg_y_offset} ${leg_z_offset}"/>
+					<origin rpy="${(offset_between_legs_wave + angle_between_legs * num) % 360 * deg2rad} 0 0" xyz="${leg_x_offset} ${leg_y_offset} ${leg_z_offset}"/>
 				</xacro:if>
 				<xacro:if value="${prefix == 'right'}">
-				<origin rpy="${-(angle_between_legs * num) % 360 * deg2rad} 0 ${pi}" xyz="${leg_x_offset} ${leg_y_offset} ${leg_z_offset}"/>
+					<origin rpy="${-(angle_between_legs * num) % 360 * deg2rad} 0 ${pi}" xyz="${leg_x_offset} ${leg_y_offset} ${leg_z_offset}"/>
 				</xacro:if>
 				<geometry>
@@ -71,22 +71,22 @@
 			</visual>
 		</link>
-<!-- /////////////// -->
+		<!-- /////////////// -->
 		<joint name="leg_${prefix}_${num}_revolute_joint" type="revolute">
-		<parent link="body"/>
+			<parent link="body"/>
 			<child link="leg_${prefix}_${num}"/>
 			<origin rpy="0       0      0" xyz="${(body_width / 4 + leg_x_offset_in_body) * side} ${first_hole_x_offset + (num) * dist_between_legs}  ${body_z_offset}"/>
 			<axis xyz="1 0  0"/>
-			<limit effort="30" lower="-1e+100" upper="1e+100" velocity="1"/>
+			<limit effort="30" lower="-1e+100" upper="1e+100" velocity="3"/>
 			<joint_properties damping="0.0" friction="0.0" />
 		</joint>
-<!-- /////////////// -->
+		<!-- /////////////// -->
 		<transmission name="leg_${prefix}_${num}_transmission">
 			<type>transmission_interface/SimpleTransmission</type>
 			<joint name="leg_${prefix}_${num}_revolute_joint">
-				<hardwareInterface>EffortJointInterface</hardwareInterface>
+				<hardwareInterface>VelocityJointInterface</hardwareInterface>
 			</joint>
 			<actuator name="leg_${prefix}_0_actuator">
-				<hardwareInterface>EffortJointInterface</hardwareInterface>
-				<mechanicalReduction>50</mechanicalReduction>
+				<hardwareInterface>VelocityJointInterface</hardwareInterface>
+				<mechanicalReduction>1</mechanicalReduction>
 			</actuator>
 		</transmission>
@@ -95,8 +95,8 @@
 	<link name="base_link"/>
 	<joint name="base_link_body_fixed" type="fixed">
-	    <parent link="base_link"/>
-	    <child link="body"/>
+		<parent link="base_link"/>
+		<child link="body"/>
 	</joint>
-<!-- /////////////// -->
+	<!-- /////////////// -->
 	<link name="body">
 		<inertial>
@@ -108,57 +108,27 @@
 				iyy="${1/12 * body_weight * (body_height * body_height + body_width * body_width)}" iyz="0"
 				izz="${1/12 * body_weight * (body_length * body_length + body_width * body_width)}" />
-		</inertial>
-		<collision >
-			<origin rpy="0  0  0" xyz="${body_x_offset} ${body_y_offset}  ${body_z_offset}"/>
-			<geometry>
-				<box size="${body_width / 2} ${body_length} ${body_height / 2}"/>
-			</geometry>
-		</collision>
-		<visual >
-			<origin rpy="0  0  0" xyz="${body_x_offset} ${body_y_offset}  ${body_z_offset}"/>
-			<geometry>
-				<box size="${body_width / 2} ${body_length} ${body_height / 2}"/>
-			</geometry>
-			<material name="green"/>
-		</visual>
-	</link>
-<!-- create needed number of legs (is implemented by recurcion) -->
-	<xacro:macro name="create_legs" params="prefix side number">
-    	<xacro:leg prefix="${prefix}" num="${number}" side="${side}"/>
-    	<xacro:if value="${number}">
-        	<xacro:create_legs number="${number-1}" prefix="${prefix}" side="${side}"/>
-    	</xacro:if>
-	</xacro:macro>
-<!-- create needed number of joints between legs (is implemented by recurcion) -->
-<!-- 	<xacro:macro name="create_dependence_between_legs" params="prefix side number">
-    			<joint name="legs_${prefix}_${number}_and_${number - 1}_revolute_joint" type="revolute">
-		<parent link="leg_${prefix}_${number}"/>
-			<child link="leg_${prefix}_${number - 1}"/>
-			<origin rpy="0       0      0" xyz="0 ${-dist_between_legs} 0"/>
-			<axis xyz="1 0  0"/>
-			<limit effort="-1" lower="-1e+100" upper="1e+100" velocity="100"/>
-		</joint>
-    	<xacro:if value="${number - 1}">
-        	<xacro:create_dependence_between_legs number="${number-1}" prefix="${prefix}" side="${side}"/>
-    	</xacro:if>
-	</xacro:macro> -->
-<xacro:create_legs prefix="left" side="1" number="${number_of_legs}" />
-<xacro:create_legs prefix="right" side="-1" number="${number_of_legs}" />
-<!-- <xacro:create_dependence_between_legs prefix="left" side="1" number="${number_of_legs}" />
-<xacro:create_dependence_between_legs prefix="right" side="-1" number="${number_of_legs}" /> -->
-<!--  <joint name="legs_l_1_and_0_revolute_joint" type="fixed">
-		<parent link="leg_left_0"/>
-			<child link="leg_left_1"/>
-			<origin rpy="0  0  0" xyz="0 ${dist_between_legs} 0"/>
-			<axis xyz="0 0  0"/>
-			<limit effort="40" lower="-1e+100" upper="1e+100" velocity="3"/>
-		</joint>
- <joint name="legs_r_1_and_0_revolute_joint" type="fixed">
-		<parent link="leg_right_0"/>
-			<child link="leg_right_1"/>
-			<origin rpy="0  0  0" xyz="0 ${dist_between_legs} 0"/>
-			<axis xyz="0 0  0"/>
-			<limit effort="40" lower="-1e+100" upper="1e+100" velocity="3"/>
-		</joint>
-  -->
-</robot>
+			</inertial>
+			<collision >
+				<origin rpy="0  0  0" xyz="${body_x_offset} ${body_y_offset}  ${body_z_offset}"/>
+				<geometry>
+					<box size="${body_width / 2} ${body_length} ${body_height / 2}"/>
+				</geometry>
+			</collision>
+			<visual >
+				<origin rpy="0  0  0" xyz="${body_x_offset} ${body_y_offset}  ${body_z_offset}"/>
+				<geometry>
+					<box size="${body_width / 2} ${body_length} ${body_height / 2}"/>
+				</geometry>
+				<material name="green"/>
+			</visual>
+		</link>
+		<!-- create needed number of legs (is implemented by recurcion) -->
+		<xacro:macro name="create_legs" params="prefix side number">
+			<xacro:leg prefix="${prefix}" num="${number}" side="${side}"/>
+			<xacro:if value="${number}">
+				<xacro:create_legs number="${number-1}" prefix="${prefix}" side="${side}"/>
+			</xacro:if>
+		</xacro:macro>
+		<xacro:create_legs prefix="left" side="1" number="${number_of_legs}" />
+		<xacro:create_legs prefix="right" side="-1" number="${number_of_legs}" />
+	</robot>

Commit message: robot work correctly, but only lower than 15 legs (15 and above - robot crashed) (60 degree)

File: strirus_robot_description/urdf/strirus.xacro (robot description, xacro)
@@ -9,5 +9,5 @@
 	<!-- number of legs need to be real number - 1 (it is from one side only)-->
 	<!-- Xacro arg provides xacro.py file.xacro real_number_of_legs:=3 -->
-	<xacro:arg name="real_number_of_legs" default="19" />
+	<xacro:arg name="real_number_of_legs" default="14" />
 	<xacro:arg name="angle_between_legs" default="60" />
 	<!-- in degree -->
@@ -27,5 +27,5 @@
 	<xacro:property name="body_width" value="${0.5 * scale}" />
 	<xacro:property name="body_height" value="${0.07 * scale}" />
-	<xacro:property name="body_weight" value="${body_width * body_length * body_height * 0.3}"/>
+	<xacro:property name="body_weight" value="${body_width * body_length * body_height * 0.2}"/>
 	<xacro:property name="leg_x_offset" value="${0 * scale}" />
 	<xacro:property name="leg_y_offset" value="${0 * scale}" />
@@ -44,5 +44,5 @@
 				<mass value="${0.05 * scale}"/>
 				<origin rpy="0  0  0" xyz="${leg_x_offset} ${leg_y_offset} ${leg_z_offset}"/>
-				<inertia ixx="0.001" ixy="0" ixz="0" iyy="0.001" iyz="0" izz="0.001"/>
+				<inertia ixx="0.000" ixy="0" ixz="0" iyy="0.000" iyz="0" izz="0.000"/>
 			</inertial>
 			<collision >
@@ -104,8 +104,9 @@
 			<mass value="${body_weight}"/>
 			<origin rpy="0  0  0" xyz="${body_x_offset} ${body_y_offset}  ${body_z_offset}"/>
-			<inertia
+<!-- 			<inertia
 				ixx="${1/12 * body_weight * (body_height * body_height + body_length * body_length)}"  ixy="0"  ixz="0"
 				iyy="${1/12 * body_weight * (body_height * body_height + body_width * body_width)}" iyz="0"
-				izz="${1/12 * body_weight * (body_length * body_length + body_width * body_width)}" />
+				izz="${1/12 * body_weight * (body_length * body_length + body_width * body_width)}" /> -->
+								<inertia ixx="0.000" ixy="0" ixz="0" iyy="0.000" iyz="0" izz="0.000"/>
 			</inertial>
 			<collision >
@@ -132,3 +133,26 @@
 		<xacro:create_legs prefix="left" side="1" number="${number_of_legs}" />
 		<xacro:create_legs prefix="right" side="-1" number="${number_of_legs}" />
-	</robot>
+		<gazebo>
+		<xacro:macro name="create_gearbox_joints_between_legs" params="prefix side number">
+			<joint name="legs_${prefix}_${number -1}_${number}_gearbox_joint" type="gearbox">
+          <parent>leg_${prefix}_${number - 1}</parent>
+          <child>leg_${prefix}_0</child>
+          <gearbox_ratio>-1</gearbox_ratio>
+          <gearbox_reference_body>base_link</gearbox_reference_body>
+          <axis>
+          	<xyz>1.000000 0.000000 0.000000</xyz>
+          	<use_parent_model_frame>true</use_parent_model_frame>
+          	</axis>
+         	<axis2>
+          		<xyz>1.000000 0.000000 0.000000</xyz>
+          		<use_parent_model_frame>true</use_parent_model_frame>
+         	 </axis2>
+      		</joint>
+      		<xacro:if value="${number - 1}">
+      			<xacro:create_gearbox_joints_between_legs number="${number-1}" prefix="${prefix}" side="${side}"/>
+      		</xacro:if>
+  			</xacro:macro>
+  			<xacro:create_gearbox_joints_between_legs prefix="left" side="1" number="${number_of_legs}" />
+			<xacro:create_gearbox_joints_between_legs prefix="right" side="-1" number="${number_of_legs}" />
+		</gazebo>
+</robot>

Commit message: Robot model is complete, add world and template for creating generate area. Add arguments for changing solver and iterations in it

File: strirus_robot_description/urdf/strirus.xacro (robot description, xacro)
@@ -9,5 +9,5 @@
 	<!-- number of legs need to be real number - 1 (it is from one side only)-->
 	<!-- Xacro arg provides xacro.py file.xacro real_number_of_legs:=3 -->
-	<xacro:arg name="real_number_of_legs" default="14" />
+	<xacro:arg name="real_number_of_legs" default="19" />
 	<xacro:arg name="angle_between_legs" default="60" />
 	<!-- in degree -->
@@ -135,7 +135,7 @@
 		<gazebo>
 		<xacro:macro name="create_gearbox_joints_between_legs" params="prefix side number">
-			<joint name="legs_${prefix}_${number -1}_${number}_gearbox_joint" type="gearbox">
-          <parent>leg_${prefix}_${number - 1}</parent>
-          <child>leg_${prefix}_0</child>
+			<joint name="legs_${prefix}_${number}_0_gearbox_joint" type="gearbox">
+          <parent>leg_${prefix}_0</parent>
+          <child>leg_${prefix}_${number}</child>
           <gearbox_ratio>-1</gearbox_ratio>
           <gearbox_reference_body>base_link</gearbox_reference_body>
