Commit message: Become possible to change all needed args only by arguments in launch file (roslaunch strirus_gazebo strirus_gazebo.launch)

File: strirus_robot_description/urdf/strirus.xacro (robot description, xacro)
@@ -8,6 +8,6 @@
 	<!-- Constants for simulating -->
 	<!-- number of legs need to be real number - 1 (it is from one side only)-->
-	<!-- Xacro arg provides xacro.py file.xacro real_number_of_legs:=3 -->
-	<xacro:arg name="real_number_of_legs" default="19" />
+	<!-- Xacro arg provides xacro.py file.xacro real_number_of_legs:=12 -->
+	<xacro:arg name="real_number_of_legs" default="12" />
 	<xacro:arg name="angle_between_legs" default="60" />
 	<!-- in degree -->
@@ -27,5 +27,5 @@
 	<xacro:property name="body_width" value="${0.5 * scale}" />
 	<xacro:property name="body_height" value="${0.07 * scale}" />
-	<xacro:property name="body_weight" value="${body_width * body_length * body_height * 0.2}"/>
+	<xacro:property name="body_weight" value="${body_width * body_length * body_height * 0.1}"/>
 	<xacro:property name="leg_x_offset" value="${0 * scale}" />
 	<xacro:property name="leg_y_offset" value="${0 * scale}" />
@@ -42,5 +42,5 @@
 		<link name="leg_${prefix}_${num}">
 			<inertial>
-				<mass value="${0.05 * scale}"/>
+				<mass value="${0.01 * scale}"/>
 				<origin rpy="0  0  0" xyz="${leg_x_offset} ${leg_y_offset} ${leg_z_offset}"/>
 				<inertia ixx="0.000" ixy="0" ixz="0" iyy="0.000" iyz="0" izz="0.000"/>
@@ -57,4 +57,31 @@
 					<mesh filename="package://strirus_robot_description/meshes/stl/leg_30_degree_normal.stl" scale="1.0 1.0 1.0"/>
 				</geometry>
+				<gazebo>
+					<surface>
+						<friction>
+							<ode>
+								<mu>0.2000</mu>
+								<mu2>0.2000</mu2>
+								<fdir1>0.000000 0.000000 0.000000</fdir1>
+								<slip1>0.000000</slip1>
+								<slip2>0.000000</slip2>
+							</ode>
+						</friction>
+						<bounce>
+							<restitution_coefficient>0.000000</restitution_coefficient>
+							<threshold>100000.000000</threshold>
+						</bounce>
+						<contact>
+							<ode>
+								<soft_cfm>0.000000</soft_cfm>
+								<soft_erp>0.200000</soft_erp>
+								<kp>100000.000000</kp>
+								<kd>1.000000</kd>
+								<max_vel>100.000000</max_vel>
+								<min_depth>0.001000</min_depth>
+							</ode>
+						</contact>
+					</surface>
+				</gazebo>
 			</collision>
 			<visual>
@@ -77,5 +104,5 @@
 			<origin rpy="0       0      0" xyz="${(body_width / 4 + leg_x_offset_in_body) * side} ${first_hole_x_offset + (num) * dist_between_legs}  ${body_z_offset}"/>
 			<axis xyz="1 0  0"/>
-			<limit effort="30" lower="-1e+100" upper="1e+100" velocity="3"/>
+			<limit effort="30" lower="-1e+100" upper="1e+100" velocity="10"/>
 			<joint_properties damping="0.0" friction="0.0" />
 		</joint>
@@ -108,5 +135,5 @@
 				iyy="${1/12 * body_weight * (body_height * body_height + body_width * body_width)}" iyz="0"
 				izz="${1/12 * body_weight * (body_length * body_length + body_width * body_width)}" /> -->
-								<inertia ixx="0.000" ixy="0" ixz="0" iyy="0.000" iyz="0" izz="0.000"/>
+				<inertia ixx="0.000" ixy="0" ixz="0" iyy="0.000" iyz="0" izz="0.000"/>
 			</inertial>
 			<collision >
@@ -134,24 +161,24 @@
 		<xacro:create_legs prefix="right" side="-1" number="${number_of_legs}" />
 		<gazebo>
-		<xacro:macro name="create_gearbox_joints_between_legs" params="prefix side number">
-			<joint name="legs_${prefix}_${number}_0_gearbox_joint" type="gearbox">
-          <parent>leg_${prefix}_0</parent>
-          <child>leg_${prefix}_${number}</child>
-          <gearbox_ratio>-1</gearbox_ratio>
-          <gearbox_reference_body>base_link</gearbox_reference_body>
-          <axis>
-          	<xyz>1.000000 0.000000 0.000000</xyz>
-          	<use_parent_model_frame>true</use_parent_model_frame>
-          	</axis>
-         	<axis2>
-          		<xyz>1.000000 0.000000 0.000000</xyz>
-          		<use_parent_model_frame>true</use_parent_model_frame>
-         	 </axis2>
-      		</joint>
-      		<xacro:if value="${number - 1}">
-      			<xacro:create_gearbox_joints_between_legs number="${number-1}" prefix="${prefix}" side="${side}"/>
-      		</xacro:if>
-  			</xacro:macro>
-  			<xacro:create_gearbox_joints_between_legs prefix="left" side="1" number="${number_of_legs}" />
+			<xacro:macro name="create_gearbox_joints_between_legs" params="prefix side number">
+				<joint name="legs_${prefix}_${number}_0_gearbox_joint" type="gearbox">
+					<parent>leg_${prefix}_0</parent>
+					<child>leg_${prefix}_${number}</child>
+					<gearbox_ratio>-1</gearbox_ratio>
+					<gearbox_reference_body>base_link</gearbox_reference_body>
+					<axis>
+						<xyz>1.000000 0.000000 0.000000</xyz>
+						<use_parent_model_frame>true</use_parent_model_frame>
+					</axis>
+					<axis2>
+						<xyz>1.000000 0.000000 0.000000</xyz>
+						<use_parent_model_frame>true</use_parent_model_frame>
+					</axis2>
+				</joint>
+				<xacro:if value="${number - 1}">
+					<xacro:create_gearbox_joints_between_legs number="${number-1}" prefix="${prefix}" side="${side}"/>
+				</xacro:if>
+			</xacro:macro>
+			<xacro:create_gearbox_joints_between_legs prefix="left" side="1" number="${number_of_legs}" />
 			<xacro:create_gearbox_joints_between_legs prefix="right" side="-1" number="${number_of_legs}" />
 		</gazebo>

Commit message: fix robot's size and mass-inertional parameters

File: strirus_robot_description/urdf/strirus.xacro (robot description, xacro)
@@ -13,6 +13,4 @@
 	<!-- in degree -->
 	<xacro:arg name="offset_between_legs_wave" default="0" />
-	<!-- scale is needed for easily change scale of stl -->
-	<xacro:property name="scale" value="5" />
 	<xacro:property name="real_number_of_legs" value="$(arg real_number_of_legs)" />
 	<xacro:property name="number_of_legs" value="${real_number_of_legs - 1}" />
@@ -21,18 +19,20 @@
 	<xacro:property name="offset_between_legs_wave" value="$(arg offset_between_legs_wave)" />
 	<!-- Body and leg Constants -->
-	<xacro:property name="body_x_offset" value="${0 * scale}" />
+	<xacro:property name="body_x_offset" value="${0}" />
 	<xacro:property name="body_y_offset" value="${body_length / 2}" />
 	<xacro:property name="body_z_offset" value="${leg_width + leg_height}" />
-	<xacro:property name="first_hole_x_offset" value="${0.05 * scale}" />
-	<xacro:property name="body_width" value="${0.5 * scale}" />
-	<xacro:property name="body_height" value="${0.07 * scale}" />
-	<xacro:property name="body_weight" value="${body_width * body_length * body_height * 0.1}"/>
-	<xacro:property name="leg_x_offset" value="${0 * scale}" />
-	<xacro:property name="leg_y_offset" value="${0 * scale}" />
-	<xacro:property name="leg_z_offset" value="${0 * scale}" />
-	<xacro:property name="leg_x_offset_in_body" value="${-0.075 * scale}" />
-	<xacro:property name="leg_width" value="${0.02 * scale}" />
-	<xacro:property name="leg_height" value="${0.08 * scale}" />
-	<xacro:property name="fallibility_between_legs" value="${(0.002 * scale) + 2 * leg_width}" />
+	<xacro:property name="first_hole_x_offset" value="${0.05}" />
+	<xacro:property name="body_width" value="${0.5}" />
+	<xacro:property name="body_height" value="${0.07}" />
+	<!-- consider that body is hollow-type , 1200 is plastic density-->
+	<xacro:property name="body_wall_thickness" value="0.01" />
+	<xacro:property name="body_weight" value="${((body_width * body_length * body_height) - ((body_width - body_wall_thickness) * (body_length - body_wall_thickness) * (body_height - body_wall_thickness))) * 1200}"/>
+	<xacro:property name="leg_x_offset" value="${0}" />
+	<xacro:property name="leg_y_offset" value="${0}" />
+	<xacro:property name="leg_z_offset" value="${0}" />
+	<xacro:property name="leg_x_offset_in_body" value="${-0.075}" />
+	<xacro:property name="leg_width" value="${0.02}" />
+	<xacro:property name="leg_height" value="${0.08}" />
+	<xacro:property name="fallibility_between_legs" value="${0.002 + 2 * leg_width}" />
 	<!-- Formulas -->
 	<xacro:property name="dist_between_legs" value="${leg_height * sin(angle_between_legs * deg2rad) + fallibility_between_legs}" />
@@ -42,7 +42,8 @@
 		<link name="leg_${prefix}_${num}">
 			<inertial>
-				<mass value="${0.01 * scale}"/>
-				<origin rpy="0  0  0" xyz="${leg_x_offset} ${leg_y_offset} ${leg_z_offset}"/>
-				<inertia ixx="0.000" ixy="0" ixz="0" iyy="0.000" iyz="0" izz="0.000"/>
+				<!-- was calcuclated in Siemens NX -->
+				<mass value="0.32"/>
+				<origin rpy="0  0  0" xyz="${leg_x_offset + 0.1} ${leg_y_offset -2.99e-7} ${leg_z_offset -0.04}"/>
+				<inertia ixx="0.0009" ixy="0" ixz="-0.0019" iyy="0.0053" iyz="0" izz="0.0044"/>
 			</inertial>
 			<collision >
@@ -55,5 +56,5 @@
 				</xacro:if>
 				<geometry>
-					<mesh filename="package://strirus_robot_description/meshes/stl/leg_30_degree_normal.stl" scale="1.0 1.0 1.0"/>
+					<mesh filename="package://strirus_robot_description/meshes/stl/leg_30_degree.stl" scale="1.0 1.0 1.0"/>
 				</geometry>
 				<gazebo>
@@ -93,5 +94,5 @@
 				</xacro:if>
 				<geometry>
-					<mesh filename="package://strirus_robot_description/meshes/stl/leg_30_degree_normal.stl" scale="1.0 1.0 1.0"/>
+					<mesh filename="package://strirus_robot_description/meshes/stl/leg_30_degree.stl" scale="1.0 1.0 1.0"/>
 				</geometry>
 				<material name="blue"/>
@@ -131,9 +132,10 @@
 			<mass value="${body_weight}"/>
 			<origin rpy="0  0  0" xyz="${body_x_offset} ${body_y_offset}  ${body_z_offset}"/>
-<!-- 			<inertia
-				ixx="${1/12 * body_weight * (body_height * body_height + body_length * body_length)}"  ixy="0"  ixz="0"
-				iyy="${1/12 * body_weight * (body_height * body_height + body_width * body_width)}" iyz="0"
-				izz="${1/12 * body_weight * (body_length * body_length + body_width * body_width)}" /> -->
-				<inertia ixx="0.000" ixy="0" ixz="0" iyy="0.000" iyz="0" izz="0.000"/>
+			<!-- consider that box is hollow-type (inertia *1.2)-->
+			<inertia
+				ixx="${1/12 * body_weight * (body_height * body_height + body_length * body_length) * 1.2}"  ixy="0"  ixz="0"
+				iyy="${1/12 * body_weight * (body_height * body_height + body_width * body_width) * 1.2}" iyz="0"
+				izz="${1/12 * body_weight * (body_length * body_length + body_width * body_width) * 1.2}" />
+<!--				<inertia ixx="0.000" ixy="0" ixz="0" iyy="0.000" iyz="0" izz="0.000"/> -->
 			</inertial>
 			<collision >

Commit message: Temporary solution for avoiding collision, by increasing solver accuracy

File: strirus_robot_description/urdf/strirus.xacro (robot description, xacro)
@@ -44,6 +44,8 @@
 				<!-- was calcuclated in Siemens NX -->
 				<mass value="0.32"/>
-				<origin rpy="0  0  0" xyz="${leg_x_offset + 0.1} ${leg_y_offset -2.99e-7} ${leg_z_offset -0.04}"/>
+				<!-- <origin rpy="0  0  0" xyz="${leg_x_offset + 0.1} ${leg_y_offset -2.99e-7} ${leg_z_offset -0.04}"/> -->
+				<origin rpy="0  0  0" xyz="0 0 0"/>
 				<inertia ixx="0.0009" ixy="0" ixz="-0.0019" iyy="0.0053" iyz="0" izz="0.0044"/>
+				<!-- <inertia ixx="0.000" ixy="0" ixz="0.00" iyy="0.00" iyz="0" izz="0.00"/> -->
 			</inertial>
 			<collision >
@@ -60,27 +62,14 @@
 				<gazebo>
 					<surface>
+						<bounce>
+							<restitution_coefficient>0.000000</restitution_coefficient> <!-- no bounce -->
+							<threshold>100000.000000</threshold>
+						</bounce>
 						<friction>
 							<ode>
-								<mu>0.2000</mu>
-								<mu2>0.2000</mu2>
-								<fdir1>0.000000 0.000000 0.000000</fdir1>
-								<slip1>0.000000</slip1>
-								<slip2>0.000000</slip2>
+								<mu>1.6</mu>
+								<mu2>1.6</mu2>
 							</ode>
 						</friction>
-						<bounce>
-							<restitution_coefficient>0.000000</restitution_coefficient>
-							<threshold>100000.000000</threshold>
-						</bounce>
-						<contact>
-							<ode>
-								<soft_cfm>0.000000</soft_cfm>
-								<soft_erp>0.200000</soft_erp>
-								<kp>100000.000000</kp>
-								<kd>1.000000</kd>
-								<max_vel>100.000000</max_vel>
-								<min_depth>0.001000</min_depth>
-							</ode>
-						</contact>
 					</surface>
 				</gazebo>
@@ -105,9 +94,9 @@
 			<origin rpy="0       0      0" xyz="${(body_width / 4 + leg_x_offset_in_body) * side} ${first_hole_x_offset + (num) * dist_between_legs}  ${body_z_offset}"/>
 			<axis xyz="1 0  0"/>
-			<limit effort="30" lower="-1e+100" upper="1e+100" velocity="10"/>
+			<limit effort="1" lower="-1e+100" upper="1e+100" velocity="1.0"/>
 			<joint_properties damping="0.0" friction="0.0" />
 		</joint>
 		<!-- /////////////// -->
-		<transmission name="leg_${prefix}_${num}_transmission">
+<!-- 		<transmission name="leg_${prefix}_${num}_transmission">
 			<type>transmission_interface/SimpleTransmission</type>
 			<joint name="leg_${prefix}_${num}_revolute_joint">
@@ -118,5 +107,8 @@
 				<mechanicalReduction>1</mechanicalReduction>
 			</actuator>
-		</transmission>
+		</transmission> -->
+	  <gazebo reference="leg_${prefix}_${num}">
+    <material>Gazebo/Gray</material>
+  </gazebo>
 	</xacro:macro>
 	<!-- Body description -->
@@ -153,4 +145,7 @@
 			</visual>
 		</link>
+		<gazebo reference="body">
+    		<material>Gazebo/DarkYellow</material>
+  		</gazebo>
 		<!-- create needed number of legs (is implemented by recurcion) -->
 		<xacro:macro name="create_legs" params="prefix side number">
@@ -164,5 +159,5 @@
 		<gazebo>
 			<xacro:macro name="create_gearbox_joints_between_legs" params="prefix side number">
-				<joint name="legs_${prefix}_${number}_0_gearbox_joint" type="gearbox">
+				<joint name="legs_${prefix}_${number}_${number-1}_gearbox_joint" type="gearbox">
 					<parent>leg_${prefix}_0</parent>
 					<child>leg_${prefix}_${number}</child>

Commit message: temp commit with needed preconditions

File: strirus_robot_description/urdf/strirus.xacro (robot description, xacro)
@@ -44,6 +44,8 @@
 				<!-- was calcuclated in Siemens NX -->
 				<mass value="0.32"/>
-				<origin rpy="0  0  0" xyz="${leg_x_offset + 0.1} ${leg_y_offset -2.99e-7} ${leg_z_offset -0.04}"/>
+				<!-- <origin rpy="0  0  0" xyz="${leg_x_offset + 0.1} ${leg_y_offset -2.99e-7} ${leg_z_offset -0.04}"/> -->
+				<origin rpy="0  0  0" xyz="0 0 0"/>
 				<inertia ixx="0.0009" ixy="0" ixz="-0.0019" iyy="0.0053" iyz="0" izz="0.0044"/>
+				<!-- <inertia ixx="0.000" ixy="0" ixz="0.00" iyy="0.00" iyz="0" izz="0.00"/> -->
 			</inertial>
 			<collision >
@@ -60,27 +62,14 @@
 				<gazebo>
 					<surface>
+						<bounce>
+							<restitution_coefficient>0.000000</restitution_coefficient> <!-- no bounce -->
+							<threshold>100000.000000</threshold>
+						</bounce>
 						<friction>
 							<ode>
-								<mu>0.2000</mu>
-								<mu2>0.2000</mu2>
-								<fdir1>0.000000 0.000000 0.000000</fdir1>
-								<slip1>0.000000</slip1>
-								<slip2>0.000000</slip2>
+								<mu>0.9</mu>
+								<mu2>0.9</mu2>
 							</ode>
 						</friction>
-						<bounce>
-							<restitution_coefficient>0.000000</restitution_coefficient>
-							<threshold>100000.000000</threshold>
-						</bounce>
-						<contact>
-							<ode>
-								<soft_cfm>0.000000</soft_cfm>
-								<soft_erp>0.200000</soft_erp>
-								<kp>100000.000000</kp>
-								<kd>1.000000</kd>
-								<max_vel>100.000000</max_vel>
-								<min_depth>0.001000</min_depth>
-							</ode>
-						</contact>
 					</surface>
 				</gazebo>
@@ -105,9 +94,9 @@
 			<origin rpy="0       0      0" xyz="${(body_width / 4 + leg_x_offset_in_body) * side} ${first_hole_x_offset + (num) * dist_between_legs}  ${body_z_offset}"/>
 			<axis xyz="1 0  0"/>
-			<limit effort="30" lower="-1e+100" upper="1e+100" velocity="10"/>
+			<limit effort="30" lower="-1e+100" upper="1e+100" velocity="1.0"/>
 			<joint_properties damping="0.0" friction="0.0" />
 		</joint>
 		<!-- /////////////// -->
-		<transmission name="leg_${prefix}_${num}_transmission">
+<!-- 		<transmission name="leg_${prefix}_${num}_transmission">
 			<type>transmission_interface/SimpleTransmission</type>
 			<joint name="leg_${prefix}_${num}_revolute_joint">
@@ -118,5 +107,8 @@
 				<mechanicalReduction>1</mechanicalReduction>
 			</actuator>
-		</transmission>
+		</transmission> -->
+	  <gazebo reference="leg_${prefix}_${num}">
+    <material>Gazebo/Gray</material>
+  </gazebo>
 	</xacro:macro>
 	<!-- Body description -->
@@ -153,4 +145,7 @@
 			</visual>
 		</link>
+		<gazebo reference="body">
+    		<material>Gazebo/DarkYellow</material>
+  		</gazebo>
 		<!-- create needed number of legs (is implemented by recurcion) -->
 		<xacro:macro name="create_legs" params="prefix side number">
@@ -164,5 +159,5 @@
 		<gazebo>
 			<xacro:macro name="create_gearbox_joints_between_legs" params="prefix side number">
-				<joint name="legs_${prefix}_${number}_0_gearbox_joint" type="gearbox">
+				<joint name="legs_${prefix}_${number}_${number-1}_gearbox_joint" type="gearbox">
 					<parent>leg_${prefix}_0</parent>
 					<child>leg_${prefix}_${number}</child>

Commit message: Fix inertial and mass center

File: strirus_robot_description/urdf/strirus.xacro (robot description, xacro)
@@ -40,38 +40,30 @@
 	<!-- Leg description -->
 	<xacro:macro name="leg" params="prefix num side">
+	<xacro:property name="angle_coeff_left" value="${(offset_between_legs_wave + angle_between_legs * num) % 360 * deg2rad}" />
+	<xacro:property name="angle_coeff_right" value="${-(angle_between_legs * num) % 360 * deg2rad}" />
 		<link name="leg_${prefix}_${num}">
 			<inertial>
 				<!-- was calcuclated in Siemens NX -->
-				<mass value="0.32"/>
-				<!-- <origin rpy="0  0  0" xyz="${leg_x_offset + 0.1} ${leg_y_offset -2.99e-7} ${leg_z_offset -0.04}"/> -->
-				<origin rpy="0  0  0" xyz="0 0 0"/>
+				<mass value="0.36"/>
+				<xacro:if value="${prefix == 'left'}">
+					<origin rpy="${angle_coeff_left} 0 0" xyz="${leg_x_offset + (0.1)} ${leg_y_offset + ((-2.99e-7 * cos(angle_coeff_left)) - (-0.04 * sin(angle_coeff_left)))} ${leg_z_offset + ( - (-2.99e-7 * sin(angle_coeff_left)) + (-0.04 * cos(angle_coeff_left)))}"/>
+				</xacro:if>
+				<xacro:if value="${prefix == 'right'}">
+					<origin rpy="${angle_coeff_right} 0 0" xyz="-${leg_x_offset + (0.1)} ${-(leg_y_offset + ((-2.99e-7 * cos(angle_coeff_right)) - (-0.04 * sin(angle_coeff_right))))} ${leg_z_offset + ( - (-2.99e-7 * sin(angle_coeff_right)) + (-0.04 * cos(angle_coeff_right)))}"/>
+				</xacro:if>
 				<inertia ixx="0.0009" ixy="0" ixz="-0.0019" iyy="0.0053" iyz="0" izz="0.0044"/>
 				<!-- <inertia ixx="0.000" ixy="0" ixz="0.00" iyy="0.00" iyz="0" izz="0.00"/> -->
 			</inertial>
-			<collision >
+			<collision>
 				<!-- legs wave offset change only on the left side -->
 				<xacro:if value="${prefix == 'left'}">
-					<origin rpy="${(offset_between_legs_wave + angle_between_legs * num) % 360 * deg2rad} 0 0" xyz="${leg_x_offset} ${leg_y_offset} ${leg_z_offset}"/>
+					<origin rpy="${angle_coeff_left} 0 0" xyz="${leg_x_offset} ${leg_y_offset} ${leg_z_offset}"/>
 				</xacro:if>
 				<xacro:if value="${prefix == 'right'}">
-					<origin rpy="${-(angle_between_legs * num) % 360 * deg2rad} 0 ${pi}" xyz="${leg_x_offset} ${leg_y_offset} ${leg_z_offset}"/>
+					<origin rpy="${angle_coeff_right} 0 ${pi}" xyz="${leg_x_offset} ${leg_y_offset} ${leg_z_offset}"/>
 				</xacro:if>
 				<geometry>
 					<mesh filename="package://strirus_robot_description/meshes/stl/leg_30_degree.stl" scale="1.0 1.0 1.0"/>
 				</geometry>
-				<gazebo>
-					<surface>
-						<bounce>
-							<restitution_coefficient>0.000000</restitution_coefficient> <!-- no bounce -->
-							<threshold>100000.000000</threshold>
-						</bounce>
-						<friction>
-							<ode>
-								<mu>0.9</mu>
-								<mu2>0.9</mu2>
-							</ode>
-						</friction>
-					</surface>
-				</gazebo>
 			</collision>
 			<visual>
@@ -94,5 +86,5 @@
 			<origin rpy="0       0      0" xyz="${(body_width / 4 + leg_x_offset_in_body) * side} ${first_hole_x_offset + (num) * dist_between_legs}  ${body_z_offset}"/>
 			<axis xyz="1 0  0"/>
-			<limit effort="30" lower="-1e+100" upper="1e+100" velocity="1.0"/>
+			<limit effort="-1" lower="-1e+100" upper="1e+100" velocity="-1"/>
 			<joint_properties damping="0.0" friction="0.0" />
 		</joint>
@@ -159,5 +151,5 @@
 		<gazebo>
 			<xacro:macro name="create_gearbox_joints_between_legs" params="prefix side number">
-				<joint name="legs_${prefix}_${number}_${number-1}_gearbox_joint" type="gearbox">
+				<joint name="legs_${prefix}_0_${number}_gearbox_joint" type="gearbox">
 					<parent>leg_${prefix}_0</parent>
 					<child>leg_${prefix}_${number}</child>
