Commit message: fix inertias problems

File: strirus_robot_description/urdf/strirus.xacro (robot description, xacro)
@@ -6,4 +6,5 @@
 	<xacro:include filename="$(find strirus_robot_description)/urdf/materials.xacro" />
 	<xacro:property name="deg2rad" value="${pi / 180}" />
+	<xacro:property name="scale" value="4" />
 	<!-- Constants for simulating -->
 	<!-- number of legs need to be real number - 1 (it is from one side only)-->
@@ -22,17 +23,17 @@
 	<xacro:property name="body_y_offset" value="${body_length / 2}" />
 	<xacro:property name="body_z_offset" value="${leg_width + leg_height}" />
-	<xacro:property name="first_hole_x_offset" value="${0.05}" />
-	<xacro:property name="body_width" value="${0.5}" />
-	<xacro:property name="body_height" value="${0.07}" />
+	<xacro:property name="first_hole_x_offset" value="${0.05 * scale}" />
+	<xacro:property name="body_width" value="${0.5  * scale}" />
+	<xacro:property name="body_height" value="${0.07  * scale}" />
 	<!-- consider that body is hollow-type , 1200 is plastic density-->
-	<xacro:property name="body_wall_thickness" value="0.01" />
+	<xacro:property name="body_wall_thickness" value="${0.01  * scale}" />
 	<xacro:property name="body_weight" value="${((body_width * body_length * body_height) - ((body_width - body_wall_thickness) * (body_length - body_wall_thickness) * (body_height - body_wall_thickness))) * 1200}"/>
 	<xacro:property name="leg_x_offset" value="${0}" />
 	<xacro:property name="leg_y_offset" value="${0}" />
 	<xacro:property name="leg_z_offset" value="${0}" />
-	<xacro:property name="leg_x_offset_in_body" value="${-0.075}" />
-	<xacro:property name="leg_width" value="${0.02}" />
-	<xacro:property name="leg_height" value="${0.08}" />
-	<xacro:property name="fallibility_between_legs" value="${0.002 + 2 * leg_width}" />
+	<xacro:property name="leg_x_offset_in_body" value="${-0.075  * scale}" />
+	<xacro:property name="leg_width" value="${0.02  * scale}" />
+	<xacro:property name="leg_height" value="${0.08  * scale}" />
+	<xacro:property name="fallibility_between_legs" value="${0.002 * scale + 2 * leg_width}" />
 	<!-- Formulas -->
 	<xacro:property name="dist_between_legs" value="${leg_height * sin(angle_between_legs * deg2rad) + fallibility_between_legs}" />
@@ -45,13 +46,12 @@
 			<inertial>
 				<!-- was calcuclated in Siemens NX -->
-				<mass value="0.36"/>
+				<mass value="${0.36 * pow(scale,3)}"/>
 				<xacro:if value="${prefix == 'left'}">
-					<origin rpy="${angle_coeff_left} 0 0" xyz="${leg_x_offset + (0.1)} ${leg_y_offset + ((-2.99e-7 * cos(angle_coeff_left)) - (-0.04 * sin(angle_coeff_left)))} ${leg_z_offset + ( - (-2.99e-7 * sin(angle_coeff_left)) + (-0.04 * cos(angle_coeff_left)))}"/>
+					<origin rpy="${angle_coeff_left} 0 0" xyz="${leg_x_offset + (0.1 * scale)} ${leg_y_offset + ((-2.99e-7 * cos(angle_coeff_left)  * scale) - (-0.04 * sin(angle_coeff_left) * scale))} ${leg_z_offset + ( - (-2.99e-7 * sin(angle_coeff_left)  * scale) + (-0.04 * cos(angle_coeff_left)  * scale))}"/>
 				</xacro:if>
 				<xacro:if value="${prefix == 'right'}">
-					<origin rpy="${angle_coeff_right} 0 0" xyz="-${leg_x_offset + (0.1)} ${-(leg_y_offset + ((-2.99e-7 * cos(angle_coeff_right)) - (-0.04 * sin(angle_coeff_right))))} ${leg_z_offset + ( - (-2.99e-7 * sin(angle_coeff_right)) + (-0.04 * cos(angle_coeff_right)))}"/>
+					<origin rpy="${angle_coeff_right} 0 0" xyz="-${leg_x_offset + (0.1 * scale)} ${-(leg_y_offset + ((-2.99e-7 * cos(angle_coeff_right) * scale) - (-0.04 * sin(angle_coeff_right) * scale)))} ${leg_z_offset + ( - (-2.99e-7 * sin(angle_coeff_right) * scale) + (-0.04 * cos(angle_coeff_right) * scale))}"/>
 				</xacro:if>
-				<inertia ixx="0.0009" ixy="0" ixz="-0.0019" iyy="0.0053" iyz="0" izz="0.0044"/>
-				<!-- <inertia ixx="0.000" ixy="0" ixz="0.00" iyy="0.00" iyz="0" izz="0.00"/> -->
+				<inertia ixx="${0.001041 * pow(scale,5)}" ixy="0" ixz="${-0.00213 * pow(scale,5)}" iyy="${0.006 * pow(scale,5)}" iyz="0" izz="${0.00497  * pow(scale,5)}"/>
 			</inertial>
 			<collision>
@@ -64,16 +64,16 @@
 				</xacro:if>
 				<geometry>
-					<mesh filename="package://strirus_robot_description/meshes/stl/leg_30_degree.stl" scale="1.0 1.0 1.0"/>
+					<mesh filename="package://strirus_robot_description/meshes/stl/leg_30_degree.stl" scale="${scale} ${scale} ${scale}"/>
 				</geometry>
 			</collision>
 			<visual>
 				<xacro:if value="${prefix == 'left'}">
-					<origin rpy="${(offset_between_legs_wave + angle_between_legs * num) % 360 * deg2rad} 0 0" xyz="${leg_x_offset} ${leg_y_offset} ${leg_z_offset}"/>
+					<origin rpy="${angle_coeff_left} 0 0" xyz="${leg_x_offset} ${leg_y_offset} ${leg_z_offset}"/>
 				</xacro:if>
 				<xacro:if value="${prefix == 'right'}">
-					<origin rpy="${-(angle_between_legs * num) % 360 * deg2rad} 0 ${pi}" xyz="${leg_x_offset} ${leg_y_offset} ${leg_z_offset}"/>
+					<origin rpy="${angle_coeff_right} 0 ${pi}" xyz="${leg_x_offset} ${leg_y_offset} ${leg_z_offset}"/>
 				</xacro:if>
 				<geometry>
-					<mesh filename="package://strirus_robot_description/meshes/stl/leg_30_degree.stl" scale="1.0 1.0 1.0"/>
+					<mesh filename="package://strirus_robot_description/meshes/stl/leg_30_degree.stl" scale="${scale} ${scale} ${scale}"/>
 				</geometry>
 				<material name="blue"/>
@@ -86,18 +86,7 @@
 			<origin rpy="0       0      0" xyz="${(body_width / 4 + leg_x_offset_in_body) * side} ${first_hole_x_offset + (num) * dist_between_legs}  ${body_z_offset}"/>
 			<axis xyz="1 0  0"/>
-			<limit effort="-1" lower="-1e+100" upper="1e+100" velocity="-1"/>
+			<limit effort="30" lower="-1e+100" upper="1e+100" velocity="3.0"/>
 			<joint_properties damping="0.0" friction="0.0" />
 		</joint>
-		<!-- /////////////// -->
-<!-- 		<transmission name="leg_${prefix}_${num}_transmission">
-			<type>transmission_interface/SimpleTransmission</type>
-			<joint name="leg_${prefix}_${num}_revolute_joint">
-				<hardwareInterface>VelocityJointInterface</hardwareInterface>
-			</joint>
-			<actuator name="leg_${prefix}_0_actuator">
-				<hardwareInterface>VelocityJointInterface</hardwareInterface>
-				<mechanicalReduction>1</mechanicalReduction>
-			</actuator>
-		</transmission> -->
 	  <gazebo reference="leg_${prefix}_${num}">
     <material>Gazebo/Gray</material>
@@ -118,8 +107,7 @@
 			<!-- consider that box is hollow-type (inertia *1.2)-->
 			<inertia
-				ixx="${1/12 * body_weight * (body_height * body_height + body_length * body_length) * 1.2}"  ixy="0"  ixz="0"
-				iyy="${1/12 * body_weight * (body_height * body_height + body_width * body_width) * 1.2}" iyz="0"
+				ixx="${1/12 * body_weight * (body_height * body_height + body_length * body_length) * 1.2 }"  ixy="0"  ixz="0"
+				iyy="${1/12 * body_weight * (body_height * body_height + body_width * body_width) * 1.2 }" iyz="0"
 				izz="${1/12 * body_weight * (body_length * body_length + body_width * body_width) * 1.2}" />
-<!--				<inertia ixx="0.000" ixy="0" ixz="0" iyy="0.000" iyz="0" izz="0.000"/> -->
 			</inertial>
 			<collision >
@@ -140,11 +128,19 @@
     		<material>Gazebo/DarkYellow</material>
   		</gazebo>
-		<!-- create needed number of legs (is implemented by recurcion) -->
-		<xacro:macro name="create_legs" params="prefix side number">
-			<xacro:leg prefix="${prefix}" num="${number}" side="${side}"/>
-			<xacro:if value="${number}">
-				<xacro:create_legs number="${number-1}" prefix="${prefix}" side="${side}"/>
-			</xacro:if>
-		</xacro:macro>
+  		<!-- create needed number of legs (is implemented by recurcion) -->
+  		<xacro:macro name="create_legs" params="prefix side number">
+  			<xacro:leg prefix="${prefix}" num="${number}" side="${side}"/>
+  			<xacro:if value="${number}">
+  				<xacro:create_legs number="${number-1}" prefix="${prefix}" side="${side}"/>
+  				<gazebo reference="leg_${prefix}_${number-1}">
+  					<mu1>0.2</mu1>
+  					<mu2>0.2</mu2>
+  				</gazebo>
+  			</xacro:if>
+  			<gazebo reference="leg_${prefix}_${number}">
+  				<mu1>0.2</mu1>
+  				<mu2>0.2</mu2>
+  			</gazebo>
+  		</xacro:macro>
 		<xacro:create_legs prefix="left" side="1" number="${number_of_legs}" />
 		<xacro:create_legs prefix="right" side="-1" number="${number_of_legs}" />

Commit message: fix model physics

File: strirus_robot_description/urdf/strirus.xacro (robot description, xacro)
@@ -2,9 +2,9 @@
 <robot name="Strirus" xmlns:xacro="http://www.ros.org/wiki/xacro">
 	<!-- Import all Gazebo-customization elements, including Gazebo colors -->
-	<xacro:include filename="$(find strirus_robot_description)/urdf/strirus.gazebo" />
+	<xacro:include filename="$(find strirus_robot_description)/urdf/strirus_plugins.gazebo" />
 	<!-- Import Rviz colors -->
 	<xacro:include filename="$(find strirus_robot_description)/urdf/materials.xacro" />
 	<xacro:property name="deg2rad" value="${pi / 180}" />
-	<xacro:property name="scale" value="4" />
+	<xacro:property name="scale" value="1" />
 	<!-- Constants for simulating -->
 	<!-- number of legs need to be real number - 1 (it is from one side only)-->
@@ -24,5 +24,5 @@
 	<xacro:property name="body_z_offset" value="${leg_width + leg_height}" />
 	<xacro:property name="first_hole_x_offset" value="${0.05 * scale}" />
-	<xacro:property name="body_width" value="${0.5  * scale}" />
+	<xacro:property name="body_width" value="${0.3  * scale}" />
 	<xacro:property name="body_height" value="${0.07  * scale}" />
 	<!-- consider that body is hollow-type , 1200 is plastic density-->
@@ -35,5 +35,5 @@
 	<xacro:property name="leg_width" value="${0.02  * scale}" />
 	<xacro:property name="leg_height" value="${0.08  * scale}" />
-	<xacro:property name="fallibility_between_legs" value="${0.002 * scale + 2 * leg_width}" />
+	<xacro:property name="fallibility_between_legs" value="${0.001 * scale + 2 * leg_width}" />
 	<!-- Formulas -->
 	<xacro:property name="dist_between_legs" value="${leg_height * sin(angle_between_legs * deg2rad) + fallibility_between_legs}" />
@@ -41,6 +41,6 @@
 	<!-- Leg description -->
 	<xacro:macro name="leg" params="prefix num side">
-	<xacro:property name="angle_coeff_left" value="${(offset_between_legs_wave + angle_between_legs * num) % 360 * deg2rad}" />
-	<xacro:property name="angle_coeff_right" value="${-(angle_between_legs * num) % 360 * deg2rad}" />
+		<xacro:property name="angle_coeff_left" value="${(offset_between_legs_wave + angle_between_legs * num) % 360 * deg2rad}" />
+		<xacro:property name="angle_coeff_right" value="${-(angle_between_legs * num) % 360 * deg2rad}" />
 		<link name="leg_${prefix}_${num}">
 			<inertial>
@@ -89,7 +89,66 @@
 			<joint_properties damping="0.0" friction="0.0" />
 		</joint>
-	  <gazebo reference="leg_${prefix}_${num}">
-    <material>Gazebo/Gray</material>
-  </gazebo>
+		<gazebo reference="leg_${prefix}_${num}">
+			<material>Gazebo/Gray</material>
+		</gazebo>
+		<gazebo reference="leg_${prefix}_${num}">
+			<collision>
+				<surface>
+					<bounce>
+						<restitution_coefficient>0</restitution_coefficient>
+						<threshold>100000</threshold>
+					</bounce>
+					<friction>
+						<ode>
+							<mu>0.5</mu>
+							<mu2>0.5</mu2>
+							<!-- <fdir1>1 0 0 </fdir1> -->
+							<slip1>0.5 </slip1>
+							<slip2>0.5 </slip2>
+						</ode>
+					</friction>
+<!-- 					<contact>
+						<ode>
+							<kp>1e+12</kp>
+							<kd>1</kd>
+							<max_vel>0.01</max_vel>
+							<soft_erp>0.2</soft_erp>
+							<soft_cfm>0</soft_cfm>
+						</ode>
+					</contact> -->
+				</surface>
+			</collision>
+		</gazebo>
+		<!-- This part for changing friction in first part of legs -->
+		<xacro:if value="${num == 0}">
+			<gazebo reference="leg_${prefix}_${num}">
+				<collision>
+					<surface>
+						<bounce>
+							<restitution_coefficient>0</restitution_coefficient>
+							<threshold>100000</threshold>
+						</bounce>
+						<friction>
+							<ode>
+								<mu>0.5</mu>
+								<mu2>0.5</mu2>
+								<!-- <fdir1>1 0 0 </fdir1> -->
+								<slip1>0.5 </slip1>
+								<slip2>0.5 </slip2>
+							</ode>
+						</friction>
+<!-- 					<contact>
+						<ode>
+							<kp>1e+12</kp>
+							<kd>1</kd>
+							<max_vel>0.01</max_vel>
+							<soft_erp>0.2</soft_erp>
+							<soft_cfm>0</soft_cfm>
+						</ode>
+					</contact> -->
+					</surface>
+				</collision>
+			</gazebo>
+		</xacro:if>
 	</xacro:macro>
 	<!-- Body description -->
@@ -110,61 +169,64 @@
 				iyy="${1/12 * body_weight * (body_height * body_height + body_width * body_width) * 1.2 }" iyz="0"
 				izz="${1/12 * body_weight * (body_length * body_length + body_width * body_width) * 1.2}" />
-			</inertial>
-			<collision >
-				<origin rpy="0  0  0" xyz="${body_x_offset} ${body_y_offset}  ${body_z_offset}"/>
-				<geometry>
-					<box size="${body_width / 2} ${body_length} ${body_height / 2}"/>
-				</geometry>
-			</collision>
-			<visual >
-				<origin rpy="0  0  0" xyz="${body_x_offset} ${body_y_offset}  ${body_z_offset}"/>
-				<geometry>
-					<box size="${body_width / 2} ${body_length} ${body_height / 2}"/>
-				</geometry>
-				<material name="green"/>
-			</visual>
-		</link>
-		<gazebo reference="body">
-    		<material>Gazebo/DarkYellow</material>
-  		</gazebo>
-  		<!-- create needed number of legs (is implemented by recurcion) -->
-  		<xacro:macro name="create_legs" params="prefix side number">
-  			<xacro:leg prefix="${prefix}" num="${number}" side="${side}"/>
-  			<xacro:if value="${number}">
-  				<xacro:create_legs number="${number-1}" prefix="${prefix}" side="${side}"/>
-  				<gazebo reference="leg_${prefix}_${number-1}">
-  					<mu1>0.2</mu1>
-  					<mu2>0.2</mu2>
-  				</gazebo>
-  			</xacro:if>
-  			<gazebo reference="leg_${prefix}_${number}">
-  				<mu1>0.2</mu1>
-  				<mu2>0.2</mu2>
-  			</gazebo>
-  		</xacro:macro>
-		<xacro:create_legs prefix="left" side="1" number="${number_of_legs}" />
-		<xacro:create_legs prefix="right" side="-1" number="${number_of_legs}" />
-		<gazebo>
-			<xacro:macro name="create_gearbox_joints_between_legs" params="prefix side number">
-				<joint name="legs_${prefix}_0_${number}_gearbox_joint" type="gearbox">
-					<parent>leg_${prefix}_0</parent>
-					<child>leg_${prefix}_${number}</child>
-					<gearbox_ratio>-1</gearbox_ratio>
-					<gearbox_reference_body>base_link</gearbox_reference_body>
-					<axis>
-						<xyz>1.000000 0.000000 0.000000</xyz>
-						<use_parent_model_frame>true</use_parent_model_frame>
-					</axis>
-					<axis2>
-						<xyz>1.000000 0.000000 0.000000</xyz>
-						<use_parent_model_frame>true</use_parent_model_frame>
-					</axis2>
-				</joint>
-				<xacro:if value="${number - 1}">
-					<xacro:create_gearbox_joints_between_legs number="${number-1}" prefix="${prefix}" side="${side}"/>
-				</xacro:if>
-			</xacro:macro>
-			<xacro:create_gearbox_joints_between_legs prefix="left" side="1" number="${number_of_legs}" />
-			<xacro:create_gearbox_joints_between_legs prefix="right" side="-1" number="${number_of_legs}" />
-		</gazebo>
+		</inertial>
+		<collision >
+			<origin rpy="0  0  0" xyz="${body_x_offset} ${body_y_offset}  ${body_z_offset}"/>
+			<geometry>
+				<box size="${body_width / 2} ${body_length} ${body_height / 2}"/>
+			</geometry>
+		</collision>
+		<visual >
+			<origin rpy="0  0  0" xyz="${body_x_offset} ${body_y_offset}  ${body_z_offset}"/>
+			<geometry>
+				<box size="${body_width / 2} ${body_length} ${body_height / 2}"/>
+			</geometry>
+			<material name="green"/>
+		</visual>
+	</link>
+	<gazebo reference="body">
+		<collision>
+			<surface>
+				<friction>
+					<ode>
+						<mu>1</mu>
+						<mu2>1</mu2>
+					</ode>
+				</friction>
+			</surface>
+		</collision>
+		<material>Gazebo/DarkYellow</material>
+	</gazebo>
+	<!-- create needed number of legs (is implemented by recurcion) -->
+	<xacro:macro name="create_legs" params="prefix side number">
+		<xacro:leg prefix="${prefix}" num="${number}" side="${side}"/>
+		<xacro:if value="${number}">
+			<xacro:create_legs number="${number-1}" prefix="${prefix}" side="${side}"/>
+		</xacro:if>
+	</xacro:macro>
+	<xacro:create_legs prefix="left" side="1" number="${number_of_legs}" />
+	<xacro:create_legs prefix="right" side="-1" number="${number_of_legs}" />
+	<gazebo>
+		<xacro:macro name="create_gearbox_joints_between_legs" params="prefix side number">
+			<joint name="legs_${prefix}_0_${number}_gearbox_joint" type="gearbox">
+				<parent>leg_${prefix}_${number-1}</parent>
+				<child>leg_${prefix}_${number}</child>
+				<gearbox_ratio>-1</gearbox_ratio>
+				<gearbox_reference_body>base_link</gearbox_reference_body>
+				<axis>
+					<xyz>1.000000 0.000000 0.000000</xyz>
+					<use_parent_model_frame>true</use_parent_model_frame>
+				</axis>
+				<axis2>
+					<xyz>1.000000 0.000000 0.000000</xyz>
+					<use_parent_model_frame>true</use_parent_model_frame>
+				</axis2>
+			</joint>
+			<!-- num -1, because gearbox joint with 0 to 0 relation is unsatisfactory -->
+			<xacro:if value="${number - 1}">
+				<xacro:create_gearbox_joints_between_legs number="${number-1}" prefix="${prefix}" side="${side}"/>
+			</xacro:if>
+		</xacro:macro>
+		<xacro:create_gearbox_joints_between_legs prefix="left" side="1" number="${number_of_legs}" />
+		<xacro:create_gearbox_joints_between_legs prefix="right" side="-1" number="${number_of_legs}" />
+	</gazebo>
 </robot>

Commit message: it is dead-end branch, but with good solutions for develop branch

File: strirus_robot_description/urdf/strirus.xacro (robot description, xacro)
@@ -1,4 +1,6 @@
 <?xml version="1.0"?>
 <robot name="Strirus" xmlns:xacro="http://www.ros.org/wiki/xacro">
+<!-- 	<xacro:arg name="namespace" default="/"/>
+	<xacro:property name="namespace" value="$(arg namespace)" /> -->
 	<xacro:property name="deg2rad" value="${pi / 180}" />
 	<xacro:property name="scale" value="1" />

Commit message: first version of omni strirus is finished

File: strirus_robot_description/urdf/strirus.xacro (robot description, xacro)
@@ -10,9 +10,11 @@
 	<xacro:arg name="real_number_of_legs" default="6" />
 	<xacro:arg name="angle_between_legs" default="60" />
+	<xacro:arg name="angle_between_body_leg" default="45" />
+	<xacro:arg name="offset_between_legs_wave" default="0" />
 	<!-- in degree -->
-	<xacro:arg name="offset_between_legs_wave" default="0" />
 	<xacro:property name="real_number_of_legs" value="$(arg real_number_of_legs)" />
 	<xacro:property name="number_of_legs" value="${real_number_of_legs - 1}" />
 	<xacro:property name="angle_between_legs" value="$(arg angle_between_legs)" />
+	<xacro:property name="angle_between_body_leg" value="$(arg angle_between_body_leg)" />
 	<!-- in degree -->
 	<xacro:property name="offset_between_legs_wave" value="$(arg offset_between_legs_wave)" />
@@ -30,7 +32,7 @@
 	<xacro:property name="leg_y_offset" value="${0}" />
 	<xacro:property name="leg_z_offset" value="${0}" />
-	<xacro:property name="leg_x_offset_in_body" value="${-0.075  * scale}" />
+	<xacro:property name="leg_x_offset_in_body" value="${-0.000  * scale}" />
 	<xacro:property name="leg_width" value="${0.02  * scale}" />
-	<xacro:property name="leg_height" value="${0.08  * scale}" />
+	<xacro:property name="leg_height" value="${0.18  * scale}" />
 	<xacro:property name="fallibility_between_legs" value="${0.001 * scale + 2 * leg_width}" />
 	<!-- Formulas -->
@@ -53,8 +55,8 @@
 				<mass value="${0.36 * pow(scale,3)}"/>
 				<xacro:if value="${prefix == 'left'}">
-					<origin rpy="${angle_coeff_left} 0 0" xyz="${leg_x_offset + (0.1 * scale)} ${leg_y_offset + ((-2.99e-7 * cos(angle_coeff_left)  * scale) - (-0.04 * sin(angle_coeff_left) * scale))} ${leg_z_offset + ( - (-2.99e-7 * sin(angle_coeff_left)  * scale) + (-0.04 * cos(angle_coeff_left)  * scale))}"/>
+					<origin rpy="${angle_coeff_left} 0 ${angle_between_body_leg * deg2rad}" xyz="${leg_x_offset + (0.1 * scale)} ${leg_y_offset + ((-2.99e-7 * cos(angle_coeff_left)  * scale) - (-0.04 * sin(angle_coeff_left) * scale))} ${leg_z_offset + ( - (-2.99e-7 * sin(angle_coeff_left)  * scale) + (-0.04 * cos(angle_coeff_left)  * scale))}"/>
 				</xacro:if>
 				<xacro:if value="${prefix == 'right'}">
-					<origin rpy="${angle_coeff_right} 0 0" xyz="-${leg_x_offset + (0.1 * scale)} ${-(leg_y_offset + ((-2.99e-7 * cos(angle_coeff_right) * scale) - (-0.04 * sin(angle_coeff_right) * scale)))} ${leg_z_offset + ( - (-2.99e-7 * sin(angle_coeff_right) * scale) + (-0.04 * cos(angle_coeff_right) * scale))}"/>
+					<origin rpy="${angle_coeff_right} 0 -${angle_between_body_leg * deg2rad}" xyz="-${leg_x_offset + (0.1 * scale)} ${-(leg_y_offset + ((-2.99e-7 * cos(angle_coeff_right) * scale) - (-0.04 * sin(angle_coeff_right) * scale)))} ${leg_z_offset + ( - (-2.99e-7 * sin(angle_coeff_right) * scale) + (-0.04 * cos(angle_coeff_right) * scale))}"/>
 				</xacro:if>
 				<inertia ixx="${0.001041 * pow(scale,5)}" ixy="0" ixz="${-0.00213 * pow(scale,5)}" iyy="${0.006 * pow(scale,5)}" iyz="0" izz="${0.00497  * pow(scale,5)}"/>
@@ -69,5 +71,5 @@
 				</xacro:if>
 				<geometry>
-					<mesh filename="package://strirus_robot_description/meshes/stl/leg_30_degree.stl" scale="${scale} ${scale} ${scale}"/>
+					<mesh filename="package://strirus_robot_description/meshes/stl/leg_strirus.stl" scale="${scale} ${scale} ${scale}"/>
 				</geometry>
 			</collision>
@@ -80,5 +82,5 @@
 				</xacro:if>
 				<geometry>
-					<mesh filename="package://strirus_robot_description/meshes/stl/leg_30_degree.stl" scale="${scale} ${scale} ${scale}"/>
+					<mesh filename="package://strirus_robot_description/meshes/stl/leg_strirus.stl" scale="${scale} ${scale} ${scale}"/>
 				</geometry>
 				<material name="blue"/>
@@ -89,5 +91,10 @@
 			<parent link="body"/>
 			<child link="leg_${prefix}_${num}"/>
-			<origin rpy="0       0      0" xyz="${(body_width / 4 + leg_x_offset_in_body) * side} ${first_hole_x_offset + (num) * dist_between_legs}  ${body_z_offset}"/>
+			<xacro:if value="${prefix == 'left'}">
+					<origin rpy="0       0      ${angle_between_body_leg * deg2rad}" xyz="${(body_width / 4 + leg_x_offset_in_body) * side} ${first_hole_x_offset + (num) * dist_between_legs}  ${body_z_offset}"/>
+				</xacro:if>
+			<xacro:if value="${prefix == 'right'}">
+					<origin rpy="0       0      ${-angle_between_body_leg * deg2rad}" xyz="${(body_width / 4 + leg_x_offset_in_body) * side} ${first_hole_x_offset + (num) * dist_between_legs}  ${body_z_offset}"/>
+				</xacro:if>
 			<axis xyz="1 0  0"/>
 			<limit effort="30" lower="-1e+100" upper="1e+100" velocity="3.0"/>
